File: PCB/KDLK24-CDD/KDLK24-CDD.kicad_sch (KiCad schematic)
At the start: 7 parts, among them J1 40PINFPC_GENERIC, U1 RA8875

Commit message: Completed schematic import
Parts:
- removed J1: 40PINFPC_GENERIC, FPC_40, symbol Connector:Conn_01x40_Socket
- removed R4, R5, R6, R7, R8: 33, RESPACK_4X0603, symbol Device:R_Pack04
- removed U1: RA8875, LQFP100, symbol Project Symbol:RA8875L3N
- added C1, C10, C11, C12, C18, C5, C6, C7, C8, C9: 0.1uF, Adafruit RA8875 TFT Breakout:0603-NO, symbol Adafruit RA8875 TFT Breakout-eagle-import:CAP_CERAMIC0603_NO
- added C16, C19, C21, C22: 10uF, Adafruit RA8875 TFT Breakout:0805-NO, symbol Adafruit RA8875 TFT Breakout-eagle-import:CAP_CERAMIC0805-NOOUTLINE
- added C17, C20, C4: 1uF, Adafruit RA8875 TFT Breakout:0805-NO, symbol Adafruit RA8875 TFT Breakout-eagle-import:CAP_CERAMIC0805-NOOUTLINE
- added C2, C3: 15pF, Adafruit RA8875 TFT Breakout:0603-NO, symbol Adafruit RA8875 TFT Breakout-eagle-import:CAP_CERAMIC0603_NO
- added D2: MBR0540, Adafruit RA8875 TFT Breakout:SOD-123, symbol Adafruit RA8875 TFT Breakout-eagle-import:DIODESOD-123
- added D3, D4: 1N4148, Adafruit RA8875 TFT Breakout:SOD-323_MINI, symbol Adafruit RA8875 TFT Breakout-eagle-import:DIODE_SOD323MINI
- added FB2: Ferrite, Adafruit RA8875 TFT Breakout:0805-NO, symbol Adafruit RA8875 TFT Breakout-eagle-import:FERRITE-0805NO
- added IC2: 741G125DBV, Adafruit RA8875 TFT Breakout:SOT23-5, symbol Adafruit RA8875 TFT Breakout-eagle-import:741G125DBV
- added J1: 40PINFPC_GENERIC, Adafruit RA8875 TFT Breakout:FPC_40, symbol Adafruit RA8875 TFT Breakout-eagle-import:40PINFPC_GENERIC
- added JP1: Breakout, Adafruit RA8875 TFT Breakout:1X15-CB, symbol Adafruit RA8875 TFT Breakout-eagle-import:PINHD-1X15-CB
- added L1: 6.8uH large inductor, Adafruit RA8875 TFT Breakout:INDUCTOR_5X5MM_NR5040_NOTHERMALS, symbol Adafruit RA8875 TFT Breakout-eagle-import:INDUCTORNR5040
- added R1: 2Ω, Adafruit RA8875 TFT Breakout:0805-NO, symbol Adafruit RA8875 TFT Breakout-eagle-import:RESISTOR0805_NOOUTLINE
- added R10, R9: 8.2Ω, Adafruit RA8875 TFT Breakout:0805-NO, symbol Adafruit RA8875 TFT Breakout-eagle-import:RESISTOR0805_NOOUTLINE
- added R11, R12: 10K, Adafruit RA8875 TFT Breakout:0603-NO, symbol Adafruit RA8875 TFT Breakout-eagle-import:RESISTOR_0603_NOOUT
- added R3: 1M, Adafruit RA8875 TFT Breakout:0603-NO, symbol Adafruit RA8875 TFT Breakout-eagle-import:RESISTOR_0603_NOOUT
- added R4, R5, R6, R7, R8: 33, Adafruit RA8875 TFT Breakout:RESPACK_4X0603, symbol Adafruit RA8875 TFT Breakout-eagle-import:RESISTOR_4PACK_US
- added SJ1: +25mA, Adafruit RA8875 TFT Breakout:SOLDERJUMPER_ARROW_NOPASTE, symbol Adafruit RA8875 TFT Breakout-eagle-import:SOLDERJUMPER
- added SJ2: +100mA, Adafruit RA8875 TFT Breakout:SOLDERJUMPER_ARROW_NOPASTE, symbol Adafruit RA8875 TFT Breakout-eagle-import:SOLDERJUMPER
- added U1: RA8875, Adafruit RA8875 TFT Breakout:LQFP100, symbol Adafruit RA8875 TFT Breakout-eagle-import:RA8875
- added U3: TPS61169, Adafruit RA8875 TFT Breakout:SC70-5, symbol Adafruit RA8875 TFT Breakout-eagle-import:VREG_BOOST_5PIN_SC70
- added U4: AP2127K-3.3, Adafruit RA8875 TFT Breakout:SOT23-5, symbol Adafruit RA8875 TFT Breakout-eagle-import:VREG_SOT23-5
- added U5: 74HC4050, Adafruit RA8875 TFT Breakout:TSSOP16, symbol Adafruit RA8875 TFT Breakout-eagle-import:74HC4050DTSSOP
- added Y1: 20MHz, Adafruit RA8875 TFT Breakout:CRYSTAL_3.2X2.5, symbol Adafruit RA8875 TFT Breakout-eagle-import:CRYSTAL3.2X2.5
Connections:
- net +24V: now also C17.1, C20.1, D2.C, J1.2 (MS)
- net +3V3: now also C11.1, C19.1, C21.1, C4.1, C5.1, C6.1, C7.1, IC2.5 (VCC), J1.4 (MS), JP1.13, R12.2, U1.13 (VDDP@1), U1.2 (OSC_VDDP), U1.25 (PS), U1.27 (SIFS1), U1.40 (VDDP@2), U1.62 (VDDP@3), U1.76 (ADC_VDD), U1.77 (RD#/EN), U1.78 (WR#/RW#), U1.79 (CS#), U1.80 (RS), U1.87 (VDDP@4), U4.5 (OUT), U5.1 (VCC)
- net 1.5V: now also C10.1, C12.1, C8.1, C9.1, U1.17 (CORE_VDD@1), U1.38 (CORE_VDD@2), U1.5 (OSC_VDD), U1.60 (LDO_OUT), U1.86 (CORE_VDD@3)
- net B3: now also J1.24 (MS), R4.5 (2)
- net B4: now also J1.25 (MS), R4.6 (2)
- net B5: now also J1.26 (MS), R4.7 (2)
- net B6: now also J1.27 (MS), R4.8 (2)
- net B7: now also J1.28 (MS), R5.5 (2)
- net DE: now also J1.34 (MS), R8.8 (2)
- net G2: now also J1.15 (MS), R5.6 (2)
- net G3: now also J1.16 (MS), R5.7 (2)
- net G4: now also J1.17 (MS), R5.8 (2)
- net G5: now also J1.18 (MS), R6.5 (2)
- net G6: now also J1.19 (MS), R6.6 (2)
- net G7: now also J1.20 (MS), R6.7 (2)
- net GND: now also C1.2, C10.2, C11.2, C12.2, C16.2, C17.2, C18.2, C19.2, C2.1, C20.2, C21.2, C22.2, C3.1, C4.2, C5.2, C6.2, C7.2, C8.2, C9.2, IC2.3 (GND), J1.13 (MS), J1.14 (MS), J1.21 (MS), J1.22 (MS), J1.23 (MS), J1.29 (MS), J1.3 (MS), J1.36 (MS), J1.5 (MS), J1.6 (MS), J1.7 (MS), JP1.14, R10.1, SJ1.1, SJ2.1, U1.1 (OSC_GNDP), U1.10 (TEST0), U1.11 (TEST1), U1.12 (TEST2), U1.16 (GND@1), U1.23 (IICA0), U1.24 (IICA1), U1.26 (GND@2), U1.28 (SIFS0), U1.33 (KIN4/GPI4), U1.34 (KIN3/GPI3), U1.35 (KIN2/GPI2), U1.36 (KIN1/GPI1), U1.37 (KIN0/GPI0), U1.39 (GND@3), U1.45 (GPIX), U1.6 (OSC_GND), U1.61 (LDO_GND), U1.70 (ADC_GND), U1.81 (C86), U1.85 (GND@4), U3.2 (GND), U4.2 (GND), U5.8 (GND)
- net HSYNC: now also J1.32 (MS), R8.5 (2)
- net INT: now also JP1.5, U1.8 (INT#)
- net LEDK: now also C18.1, J1.1 (MSV), R1.2, R10.2, R9.2, U3.3 (FB)
- net MOSI_3V: now also U1.43 (SDI/SDA), U5.4 (2Y)
- net PIXCLK: now also J1.30 (MS), R8.7 (2)
- net PWM0: now also D3.C, U1.14 (PWM1)
- net R3: now also J1.8 (MS), R6.8 (2)
- net R4: now also J1.9 (MS), R7.5 (2)
- net R5: now also J1.10 (MS), R7.6 (2)
- net R6: now also J1.11 (MS), R7.7 (2)
- net R7: now also J1.12 (MS), R7.8 (2)
- net RA_MISO: now also IC2.2 (I), U1.42 (SDO)
- net RESET_3V: now also U1.9 (RST#), U5.10 (4Y)
- net SPI_CLK_3V: now also U1.44 (SCL), U5.2 (1Y)
- net SPI_CS_3V: now also IC2.1 (OE), U1.41 (SCS#), U5.6 (3Y)
- net VSYNC: now also J1.33 (MS), R8.6 (2)
- net WAIT: now also JP1.6, U1.7 (WAIT#)
- net X+: now also J1.37 (MS), JP1.1, U1.75 (XP)
- net X-: now also J1.39 (MS), JP1.2, U1.72 (XN)
- net Y+: now also J1.38 (MS), JP1.4, U1.73 (YP)
- net Y-: now also J1.40 (MS), JP1.3, U1.74 (YN)
- new net: R5.4 (1), U1.55 (PDAT4)
- new net: R4.1, U1.54 (PDAT3)
- new net: R5.2 (1), U1.57 (PDAT6)
- new net: R5.1, U1.58 (PDAT7)
- new net: R7.1, U1.69 (PDAT15)
- new net: C22.1, FB2.1 (P$1), U4.1 (IN), U4.3 (EN)
- new net: R7.2 (1), U1.68 (PDAT14)
- new net: D2.A, L1.P$2 (2), U3.1 (SW)
- new net: C3.2, R3.1, U1.4 (XO), Y1.1
- new net: D3.A, D4.A, R11.1, U3.4 (SHDN)
- new net: C1.1, U1.71 (ADC_VREF)
- new net: R9.1, SJ1.2
- new net: R6.4 (1), U1.59 (PDAT8)
- new net: R4.3 (1), U1.52 (PDAT1)
- new net: R4.2 (1), U1.53 (PDAT2)
- new net: R1.1, SJ2.2
- new net: R8.3 (1), U1.48 (VSYNC)
- new net: R6.1, U1.65 (PDAT11)
- new net: C2.2, R3.2, U1.3 (XI), Y1.2
- new net: R8.2 (1), U1.49 (PCLK)
- new net: R8.4 (1), U1.47 (HSYNC)
- new net: R6.2 (1), U1.64 (PDAT10)
- new net: R7.3 (1), U1.67 (PDAT13)
- new net: R7.4 (1), U1.66 (PDAT12)
- new net: R6.3 (1), U1.63 (PDAT9)
- new net: R8.1, U1.50 (DE)
- new net: R4.4 (1), U1.51 (PDAT0)
- new net: R5.3 (1), U1.56 (PDAT5)
- new net BACKLITE: D4.C, JP1.12
- new net CS: JP1.8, U5.7 (3A)
- new net MISO: IC2.4 (O), JP1.10
- new net MOSI: JP1.9, U5.5 (2A)
- new net ON/OFF: J1.31 (MS), U1.46 (GPOX)
- new net RESET: JP1.7, R12.1, U5.9 (4A)
- new net SCK: JP1.11, U5.3 (1A)
- new net VIN: C16.1, FB2.2 (P$2), JP1.15, L1.P$1 (1), R11.2, U3.5 (VIN)
Other:
- note added: "3.3V Regulation"
- note added: "7 x 3.2V LED boost"
